File: _autosave-HammerHacks II Badge PCB.kicad_pcb (KiCad board)
At the start: 2 copper layers, 44.5 x 44.5 mm, 5 parts

Commit message: rough
Parts:
- moved R2 1.48 mm to (138.1, 111.9)
Routing:
- net Net-(BT1-+): track 0.00 -> 51.3 mm
- net Net-(BT1--): track 0.00 -> 42.3 mm, vias 0 -> 1
- net Net-(D1-A): track 0.00 -> 8.07 mm
- net Net-(D2-A): track 0.00 -> 6.75 mm
Other:
- outline, holes or cut-outs redrawn
